File: gpio_extend/gpi.kicad_sch (KiCad schematic)
At the start: 12 parts, among them J16 Conn_01x09_Socket, J17 Conn_01x03_Pin, U7 74HC165

Commit message: Final for production
Parts:
- R57: renamed from R33; footprint Capacitor_SMD:C_0603_1608Metric_Pad1.08x0.95mm_HandSolder -> Resistor_SMD:R_0603_1608Metric_Pad0.98x0.95mm_HandSolder
- R58: renamed from R34; footprint Capacitor_SMD:C_0603_1608Metric_Pad1.08x0.95mm_HandSolder -> Resistor_SMD:R_0603_1608Metric_Pad0.98x0.95mm_HandSolder
- R59: renamed from R35; footprint Capacitor_SMD:C_0603_1608Metric_Pad1.08x0.95mm_HandSolder -> Resistor_SMD:R_0603_1608Metric_Pad0.98x0.95mm_HandSolder
- R60: renamed from R36; footprint Capacitor_SMD:C_0603_1608Metric_Pad1.08x0.95mm_HandSolder -> Resistor_SMD:R_0603_1608Metric_Pad0.98x0.95mm_HandSolder
- R61: renamed from R37; footprint Capacitor_SMD:C_0603_1608Metric_Pad1.08x0.95mm_HandSolder -> Resistor_SMD:R_0603_1608Metric_Pad0.98x0.95mm_HandSolder
- R62: renamed from R38; footprint Capacitor_SMD:C_0603_1608Metric_Pad1.08x0.95mm_HandSolder -> Resistor_SMD:R_0603_1608Metric_Pad0.98x0.95mm_HandSolder
- R63: renamed from R39; footprint Capacitor_SMD:C_0603_1608Metric_Pad1.08x0.95mm_HandSolder -> Resistor_SMD:R_0603_1608Metric_Pad0.98x0.95mm_HandSolder
- R64: renamed from R48; footprint Capacitor_SMD:C_0603_1608Metric_Pad1.08x0.95mm_HandSolder -> Resistor_SMD:R_0603_1608Metric_Pad0.98x0.95mm_HandSolder
- renumbered C6 to C9, J16 to J20, J17 to J21, U7 to U9
Connections:
- no-connect marks 0 -> 1
Changed lines of the file:
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@@
 		(color 0 0 0 0)
 	)
+	(no_connect
+		(at 153.67 81.28)
+	)
 	(wire
 		(pts
@@
 		)
 	)
-	(text "Note: The register is used in reverse. D7 is LSB and D0 is MSB.\n"
+	(text "Note: \nThe register is used in reverse.\nD7 is LSB and D0 is MSB.\n"
 		(exclude_from_sim no)
-		(at 97.028 68.072 0)
+		(at 119.126 69.342 0)
 		(effects
 			(font
@@
 		(shape input)
 		(at 125.73 78.74 180)
-		(fields_autoplaced yes)
 		(effects
 			(font
@@
 		(shape input)
 		(at 125.73 104.14 180)
-		(fields_autoplaced yes)
 		(effects
 			(font
@@
 		(shape input)
 		(at 125.73 109.22 180)
-		(fields_autoplaced yes)
 		(effects
 			(font
@@
 		(shape output)
 		(at 160.02 78.74 0)
-		(fields_autoplaced yes)
 		(effects
 			(font
@@
 		(dnp no)
 		(fields_autoplaced yes)
-		(property "Reference" "#PWR0107"
+		(property "Reference" "#PWR0112"
 			(at 140.97 63.5 0)
 			(effects
@@
 		(dnp no)
 		(fields_autoplaced yes)
-		(property "Reference" "#PWR0105"
+		(property "Reference" "#PWR0110"
 			(at 181.61 115.57 0)
 			(effects
@@
 		(dnp no)
 		(fields_autoplaced yes)
-		(property "Reference" "C6"
+		(property "Reference" "C9"
 			(at 185.42 96.5199 0)
 			(effects
@@
 			(project "gpio_extend"
 				(path "/e8989d35-7e4b-48bc-9b5c-be413cedaeca/8b451107-a402-4b7b-a8c5-0b64d69416de"
+					(reference "C9")
+					(unit 1)
+				)
+				(path "/e8989d35-7e4b-48bc-9b5c-be413cedaeca/b318149f-8885-4a20-9a5f-bc0269ae6c02"
+					(reference "C6")
+					(unit 1)
+				)
+				(path "/e8989d35-7e4b-48bc-9b5c-be413cedaeca/b9eb6ae7-ff70-445a-813e-698efd1ba647"
 					(reference "C8")
 					(unit 1)
 				)
-				(path "/e8989d35-7e4b-48bc-9b5c-be413cedaeca/b318149f-8885-4a20-9a5f-bc0269ae6c02"
-					(reference "C5")
-					(unit 1)
-				)
-				(path "/e8989d35-7e4b-48bc-9b5c-be413cedaeca/b9eb6ae7-ff70-445a-813e-698efd1ba647"
+				(path "/e8989d35-7e4b-48bc-9b5c-be413cedaeca/bd735a6f-214d-4695-a15e-b779d348a5fa"
 					(reference "C7")
-					(unit 1)
-				)
-				(path "/e8989d35-7e4b-48bc-9b5c-be413cedaeca/bd735a6f-214d-4695-a15e-b779d348a5fa"
-					(reference "C6")
 					(unit 1)
 				)
@@
 		(on_board yes)
 		(dnp no)
-		(property "Reference" "R33"
+		(property "Reference" "R57"
 			(at 110.744 107.188 90)
 			(effects
@@
 			)
 		)
-		(property "Footprint" "Capacitor_SMD:C_0603_1608Metric_Pad1.08x0.95mm_HandSolder"
+		(property "Footprint" "Resistor_SMD:R_0603_1608Metric_Pad0.98x0.95mm_HandSolder"
 			(at 111.252 105.41 90)
 			(effects
@@
 		(on_board yes)
 		(dnp no)
-		(property "Reference" "R34"
+		(property "Reference" "R58"
 			(at 105.664 107.188 90)
 			(effects
@@
 			)
 		)
-		(property "Footprint" "Capacitor_SMD:C_0603_1608Metric_Pad1.08x0.95mm_HandSolder"
+		(property "Footprint" "Resistor_SMD:R_0603_1608Metric_Pad0.98x0.95mm_HandSolder"
 			(at 106.172 105.41 90)
 			(effects
@@
 		(on_board yes)
 		(dnp no)
-		(property "Reference" "R37"
+		(property "Reference" "R61"
 			(at 90.424 107.188 90)
 			(effects
@@
 			)
 		)
-		(property "Footprint" "Capacitor_SMD:C_0603_1608Metric_Pad1.08x0.95mm_HandSolder"
+		(property "Footprint" "Resistor_SMD:R_0603_1608Metric_Pad0.98x0.95mm_HandSolder"
 			(at 90.932 105.41 90)
 			(effects
@@
 		(on_board yes)
 		(dnp no)
-		(property "Reference" "J17"
+		(property "Reference" "J21"
 			(at 61.468 109.474 0)
 			(effects
@@
 		(on_board yes)
 		(dnp no)
-		(property "Reference" "J16"
+		(property "Reference" "J20"
 			(at 48.514 81.788 0)
 			(effects
@@
 		(on_board yes)
 		(dnp no)
-		(property "Reference" "R39"
+		(property "Reference" "R63"
 			(at 80.264 107.188 90)
 			(effects
@@
 			)
 		)
-		(property "Footprint" "Capacitor_SMD:C_0603_1608Metric_Pad1.08x0.95mm_HandSolder"
+		(property "Footprint" "Resistor_SMD:R_0603_1608Metric_Pad0.98x0.95mm_HandSolder"
 			(at 80.772 105.41 90)
 			(effects
@@
 		(dnp no)
 		(fields_autoplaced yes)
-		(property "Reference" "#PWR0104"
+		(property "Reference" "#PWR0109"
 			(at 140.97 133.35 0)
 			(effects
@@
 		(on_board yes)
 		(dnp no)
-		(property "Reference" "#PWR0106"
+		(property "Reference" "#PWR0111"
 			(at 181.61 90.17 0)
 			(effects
@@
 		(on_board yes)
 		(dnp no)
-		(property "Reference" "R38"
+		(property "Reference" "R62"
 			(at 85.344 107.188 90)
 			(effects
@@
 			)
 		)
-		(property "Footprint" "Capacitor_SMD:C_0603_1608Metric_Pad1.08x0.95mm_HandSolder"
+		(property "Footprint" "Resistor_SMD:R_0603_1608Metric_Pad0.98x0.95mm_HandSolder"
 			(at 85.852 105.41 90)
 			(effects
@@
 		(on_board yes)
 		(dnp no)
-		(property "Reference" "R35"
+		(property "Reference" "R59"
 			(at 100.584 107.188 90)
 			(effects
@@
 			)
 		)
-		(property "Footprint" "Capacitor_SMD:C_0603_1608Metric_Pad1.08x0.95mm_HandSolder"
+		(property "Footprint" "Resistor_SMD:R_0603_1608Metric_Pad0.98x0.95mm_HandSolder"
 			(at 101.092 105.41 90)
 			(effects
@@
 		(dnp no)
 		(fields_autoplaced yes)
-		(property "Reference" "U7"
+		(property "Reference" "U9"
 			(at 143.1641 71.12 0)
 			(effects
@@
 		(on_board yes)
 		(dnp no)
-		(property "Reference" "R48"
+		(property "Reference" "R64"
 			(at 75.184 107.188 90)
 			(effects
@@
 			)
 		)
-		(property "Footprint" "Capacitor_SMD:C_0603_1608Metric_Pad1.08x0.95mm_HandSolder"
+		(property "Footprint" "Resistor_SMD:R_0603_1608Metric_Pad0.98x0.95mm_HandSolder"
 			(at 75.692 105.41 90)
 			(effects
@@
 		(dnp no)
 		(fields_autoplaced yes)
-		(property "Reference" "#PWR0103"
+		(property "Reference" "#PWR0108"
 			(at 69.85 110.49 0)
 			(effects
@@
 		(on_board yes)
 		(dnp no)
-		(property "Reference" "R36"
+		(property "Reference" "R60"
 			(at 95.504 107.188 90)
 			(effects
@@
 			)
 		)
-		(property "Footprint" "Capacitor_SMD:C_0603_1608Metric_Pad1.08x0.95mm_HandSolder"
+		(property "Footprint" "Resistor_SMD:R_0603_1608Metric_Pad0.98x0.95mm_HandSolder"
 			(at 96.012 105.41 90)
 			(effects
