File: gpio_extend/gpio_extend.kicad_pcb (KiCad board)
At the start: 2 copper layers, 88 x 65 mm, 138 parts, among them J1 Conn_01x07_Socket, J10 Conn_01x10_Socket, J11 Conn_01x02_Pin, J12 Conn_01x11_Socket, J13 Conn_01x10_Socket, J14 Conn_01x09_Socket, J15 Conn_01x03_Pin, J16 Conn_01x09_Socket, J17 Conn_01x03_Pin, J18 Conn_01x09_Socket, J19 Conn_01x03_Pin, J2 Conn_01x02_Pin, J20 Conn_01x09_Socket, J21 Conn_01x03_Pin, J3 Conn_01x11_Socket, J4 Conn_01x10_Socket, J5 Conn_01x02_Pin, J6 Conn_01x11_Socket, J7 Conn_01x10_Socket, J8 Conn_01x02_Pin, J9 Conn_01x11_Socket, U1 74AC595, U2 74AC595, U3 74AC595, U4 74AC595, U5 74AHC1G00, U6 74HC165, U7 74HC165, U8 74HC165, U9 74HC165

Commit message: Final for production
Parts:
- added C5: 0.1uF, Capacitor_SMD:C_0603_1608Metric_Pad1.08x0.95mm_HandSolder, F.Cu at (145.5, 67.2)
- added J22: Conn_01x07_Socket, Connector_PinSocket_2.54mm:PinSocket_1x07_P2.54mm_Vertical, F.Cu at (154.6, 112.3)
- R33, R34, R35, R36, R37, R38, R39, R40, R41, R42, R43, R44, R45, R46, R47, R48, R49, R50, R51, R52, R53, R54, R55, R56, R57, R58, R59, R60, R61, R62, R63, R64: footprint Capacitor_SMD:C_0603_1608Metric_Pad1.08x0.95mm_HandSolder -> Resistor_SMD:R_0603_1608Metric_Pad0.98x0.95mm_HandSolder
- renumbered C5 to C6, C6 to C7, C7 to C8, C8 to C9
Connections:
- U1 pad 10: /gpo0/n_clr -> VCC
- U1 pad 13: /gpo0/n_oe -> GND
- U2 pad 10: /gpo1/n_clr -> VCC
- U2 pad 13: /gpo1/n_oe -> GND
- U3 pad 10: /gpo2/n_clr -> VCC
- U3 pad 13: /gpo2/n_oe -> GND
- U4 pad 10: /gpo3/n_clr -> VCC
- U4 pad 13: /gpo3/n_oe -> GND
Routing:
- net GND: track 429.8 -> 515.4 mm, vias 8 -> 25
- net VCC: track 264.1 -> 292.4 mm
- net /gpi3/ser_in: track 1.76 -> 15.9 mm
- net /gpo0/pclk: track 83.4 -> 95.4 mm
- net /gpo3/ser_out: track 0.00 -> 9.80 mm
- net /gpi0/clk: track 103.2 -> 111.4 mm
- net Net-(D17-A): track 15.2 -> 17.8 mm
- net Net-(D17-K): track 0.00 -> 2.06 mm
- added copper zone on B.Cu, net GND
- added copper zone on F.Cu, net GND
