File: gpio_extend/gpio_extend.kicad_sch (KiCad schematic)
At the start: 6 parts, among them J1 Conn_01x07_Socket, U5 74AHC1G00

Commit message: Final for production
Parts:
- added C5: 0.1uF, Capacitor_SMD:C_0603_1608Metric_Pad1.08x0.95mm_HandSolder, symbol Device:C
- added J22: Conn_01x07_Socket, Connector_PinSocket_2.54mm:PinSocket_1x07_P2.54mm_Vertical, symbol Connector:Conn_01x07_Socket
Connections:
- net GND: now also C5.2, J22.1 (Pin_1), J22.7 (Pin_7)
- net VCC: now also C5.1, J22.6 (Pin_6)
- net gpi0/clk: now also J22.3 (Pin_3)
- net gpi3/ser_in: now also J22.5 (Pin_5)
- net gpo0/pclk: now also J22.2 (Pin_2)
- net gpo3/ser_out: now also J22.4 (Pin_4)
Other:
- note added: "Possible extension for more than 32 bit in/out."
- moved on the sheet: J1
