File: gpio_extend/gpo.kicad_sch (KiCad schematic)
At the start: 21 parts, among them J5 Conn_01x02_Pin, J6 Conn_01x11_Socket, J7 Conn_01x10_Socket, U2 74AC595

Commit message: Final for production
Parts:
- renumbered C1 to C2
Other:
- note added: "This should be an 8-bit R2R ladder. But I couldn't find a symbol. Therfore a DNP pin header with same footprint. Sorry, it's the first time I try out KiCad."
- note removed: "This should be an 8-bit R2R ladder. But I couldn't find a symbol. Therfore a DNP pin header with same footprint."
- moved on the sheet: J7
Changed lines of the file:
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@@
 	(wire
 		(pts
-			(xy 133.35 83.82) (xy 154.94 83.82)
+			(xy 133.35 83.82) (xy 158.75 83.82)
 		)
 		(stroke
@@
 	(wire
 		(pts
-			(xy 128.27 86.36) (xy 152.4 86.36)
-		)
-		(stroke
-			(width 0)
-			(type default)
-		)
-	)
-	(wire
-		(pts
-			(xy 147.32 91.44) (xy 147.32 71.12)
+			(xy 128.27 86.36) (xy 156.21 86.36)
+		)
+		(stroke
+			(width 0)
+			(type default)
+		)
+	)
+	(wire
+		(pts
+			(xy 151.13 91.44) (xy 151.13 71.12)
 		)
 		(stroke
@@
 	(wire
 		(pts
-			(xy 123.19 88.9) (xy 149.86 88.9)
+			(xy 123.19 88.9) (xy 153.67 88.9)
 		)
 		(stroke
@@
 	(wire
 		(pts
-			(xy 154.94 83.82) (xy 154.94 71.12)
+			(xy 158.75 83.82) (xy 158.75 71.12)
 		)
 		(stroke
@@
 	(wire
 		(pts
-			(xy 160.02 78.74) (xy 160.02 71.12)
-		)
-		(stroke
-			(width 0)
-			(type default)
-		)
-	)
-	(wire
-		(pts
-			(xy 139.7 73.66) (xy 139.7 71.12)
+			(xy 163.83 78.74) (xy 163.83 71.12)
+		)
+		(stroke
+			(width 0)
+			(type default)
+		)
+	)
+	(wire
+		(pts
+			(xy 143.51 73.66) (xy 143.51 71.12)
 		)
 		(stroke
@@
 	(wire
 		(pts
-			(xy 152.4 86.36) (xy 152.4 71.12)
+			(xy 156.21 86.36) (xy 156.21 71.12)
 		)
 		(stroke
@@
 	(wire
 		(pts
-			(xy 118.11 91.44) (xy 147.32 91.44)
+			(xy 118.11 91.44) (xy 151.13 91.44)
 		)
 		(stroke
@@
 	(wire
 		(pts
-			(xy 104.14 73.66) (xy 139.7 73.66)
-		)
-		(stroke
-			(width 0)
-			(type default)
-		)
-	)
-	(wire
-		(pts
-			(xy 157.48 81.28) (xy 157.48 71.12)
-		)
-		(stroke
-			(width 0)
-			(type default)
-		)
-	)
-	(wire
-		(pts
-			(xy 138.43 81.28) (xy 157.48 81.28)
+			(xy 104.14 73.66) (xy 143.51 73.66)
+		)
+		(stroke
+			(width 0)
+			(type default)
+		)
+	)
+	(wire
+		(pts
+			(xy 161.29 81.28) (xy 161.29 71.12)
+		)
+		(stroke
+			(width 0)
+			(type default)
+		)
+	)
+	(wire
+		(pts
+			(xy 138.43 81.28) (xy 161.29 81.28)
 		)
 		(stroke
@@
 	(wire
 		(pts
-			(xy 149.86 88.9) (xy 149.86 71.12)
+			(xy 153.67 88.9) (xy 153.67 71.12)
 		)
 		(stroke
@@
 	(wire
 		(pts
-			(xy 142.24 96.52) (xy 142.24 71.12)
-		)
-		(stroke
-			(width 0)
-			(type default)
-		)
-	)
-	(wire
-		(pts
-			(xy 107.95 96.52) (xy 142.24 96.52)
+			(xy 146.05 96.52) (xy 146.05 71.12)
+		)
+		(stroke
+			(width 0)
+			(type default)
+		)
+	)
+	(wire
+		(pts
+			(xy 107.95 96.52) (xy 146.05 96.52)
 		)
 		(stroke
@@
 	(wire
 		(pts
-			(xy 162.56 76.2) (xy 162.56 71.12)
-		)
-		(stroke
-			(width 0)
-			(type default)
-		)
-	)
-	(wire
-		(pts
-			(xy 113.03 93.98) (xy 144.78 93.98)
+			(xy 166.37 76.2) (xy 166.37 71.12)
+		)
+		(stroke
+			(width 0)
+			(type default)
+		)
+	)
+	(wire
+		(pts
+			(xy 113.03 93.98) (xy 148.59 93.98)
 		)
 		(stroke
@@
 	(wire
 		(pts
-			(xy 127 76.2) (xy 162.56 76.2)
-		)
-		(stroke
-			(width 0)
-			(type default)
-		)
-	)
-	(wire
-		(pts
-			(xy 143.51 78.74) (xy 160.02 78.74)
+			(xy 127 76.2) (xy 166.37 76.2)
+		)
+		(stroke
+			(width 0)
+			(type default)
+		)
+	)
+	(wire
+		(pts
+			(xy 143.51 78.74) (xy 163.83 78.74)
 		)
 		(stroke
@@
 	(wire
 		(pts
-			(xy 144.78 93.98) (xy 144.78 71.12)
+			(xy 148.59 93.98) (xy 148.59 71.12)
 		)
 		(stroke
@@
 		)
 	)
-	(text "This should be an 8-bit R2R ladder.\nBut I couldn't find a symbol.\nTherfore a DNP pin header with same footprint."
+	(text "This should be an 8-bit R2R ladder.\nBut I couldn't find a symbol.\nTherfore a DNP pin header with same footprint.\nSorry, it's the first time I try out KiCad."
 		(exclude_from_sim no)
 		(at 157.734 58.42 0)
@@
 		(shape input)
 		(at 63.5 93.98 180)
-		(fields_autoplaced yes)
 		(effects
 			(font
@@
 		(shape input)
 		(at 63.5 107.95 180)
-		(fields_autoplaced yes)
 		(effects
 			(font
@@
 		(shape input)
 		(at 63.5 78.74 180)
-		(fields_autoplaced yes)
 		(effects
 			(font
@@
 		(shape input)
 		(at 63.5 83.82 180)
-		(fields_autoplaced yes)
 		(effects
 			(font
@@
 		(shape input)
 		(at 63.5 86.36 180)
-		(fields_autoplaced yes)
 		(effects
 			(font
@@
 		(shape input)
 		(at 63.5 91.44 180)
-		(fields_autoplaced yes)
 		(effects
 			(font
@@
 		(dnp no)
 		(fields_autoplaced yes)
-		(property "Reference" "#PWR013"
+		(property "Reference" "#PWR014"
 			(at 193.04 101.6 0)
 			(effects
@@
 		(dnp no)
 		(fields_autoplaced yes)
-		(property "Reference" "#PWR09"
+		(property "Reference" "#PWR010"
 			(at 193.04 86.36 0)
 			(effects
@@
 	(symbol
 		(lib_id "Connector:Conn_01x10_Socket")
-		(at 152.4 66.04 270)
+		(at 156.21 66.04 270)
 		(mirror x)
 		(unit 1)
@@
 		(dnp yes)
 		(property "Reference" "J7"
-			(at 151.638 64.008 90)
+			(at 155.448 64.008 90)
 			(effects
 				(font
@@
 		)
 		(property "Value" "Conn_01x10_Socket"
-			(at 151.13 63.5 90)
+			(at 154.94 63.5 90)
 			(effects
 				(font
@@
 		)
 		(property "Footprint" "Connector_PinSocket_2.54mm:PinSocket_1x10_P2.54mm_Vertical"
-			(at 152.4 66.04 0)
+			(at 156.21 66.04 0)
 			(effects
 				(font
@@
 		)
 		(property "Datasheet" "~"
-			(at 152.4 66.04 0)
+			(at 156.21 66.04 0)
 			(effects
 				(font
@@
 		)
 		(property "Description" "Generic connector, single row, 01x10, script generated"
-			(at 152.4 66.04 0)
+			(at 156.21 66.04 0)
 			(effects
 				(font
@@
 		(dnp no)
 		(fields_autoplaced yes)
-		(property "Reference" "C1"
+		(property "Reference" "C2"
 			(at 196.85 87.6299 0)
 			(effects
